File: KiCad/HexDisplay.kicad_sch (KiCad schematic)
At the start: 27 parts, among them J1 Data_In, U1 ATmega328-P, U2 74HCT574, U3 D148K, U4 D148K, Y1 16MHz

Commit message: Updates of KiCad files and README
Parts:
- J1: OrderInfo (none) -> https://www.digikey.com/en/products/detail/harwin-inc/M20-9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
Changed lines of the file:
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@@
 			)
 		)
-		(property "OrderInfo" ""
+		(property "OrderInfo" "https://www.digikey.com/en/products/detail/harwin-inc/M20-9771146/3920928"
 			(at 36.83 160.02 0)
 			(effects
@@
 					(size 1.27 1.27)
 				)
+				(hide yes)
 			)
 		)
